Commit message: spelling correction in robot joint

File: urdf/iam_bot.urdf (robot description, URDF)
Before this commit: robot iam_bot, 8 links, 7 joints
Joints:
- removed joint bight_caster_Revolute
- added joint right_caster_Revolute: type continuous, parent base_link, child right_caster_connector, origin xyz=-0.20483935 0.06500879000000001 0.02858005 rpy=0.0 -0.0 0.0, axis 0.0 0.0 1.0
