Commit message: rviz implementation

File: iam_bot/urdf/iam_bot.urdf (robot description, URDF)
Before this commit: robot iam_bot, 8 links, 7 joints
Links:
- link base_link: geometry collision mesh filename=package://iam_bot/meshes/base_link_col.stl scale=0.001 0.001 0.001; visual mesh filename=package://iam_bot/meshes/base_link.stl scale=0.001 0.001 0.001
- link left_caster_connector: geometry collision box size=0.01 0.02 0.01; visual mesh filename=package://iam_bot/meshes/left_caster_connector.stl scale=0.001 0.001 0.001
- link left_caster_wheel: geometry collision cylinder length=0.01 radius=0.011; visual mesh filename=package://iam_bot/meshes/left_caster_wheel.stl scale=0.001 0.001 0.001
- link left_wheel: geometry collision cylinder length=0.055 radius=0.053; visual mesh filename=package://iam_bot/meshes/left_wheel.stl scale=0.001 0.001 0.001
- link right_caster_connector: geometry collision box size=0.01 0.02 0.01; visual mesh filename=package://iam_bot/meshes/right_caster_connector.stl scale=0.001 0.001 0.001
- link right_caster_wheel: geometry collision cylinder length=0.01 radius=0.011; visual mesh filename=package://iam_bot/meshes/right_caster_wheel.stl scale=0.001 0.001 0.001
- link right_wheel: geometry collision cylinder length=0.055 radius=0.053; visual mesh filename=package://iam_bot/meshes/right_wheel.stl scale=0.001 0.001 0.001
- link top_lidar_sensor: geometry collision box size=0.12 0.072 0.055; visual mesh filename=package://iam_bot/meshes/top_lidar_sensor.stl scale=0.001 0.001 0.001

Commit message: facial recognition and camera implementation

File: iam_bot/urdf/iam_bot.urdf (robot description, URDF)
Before this commit: robot iam_bot, 8 links, 7 joints
Links:
- added link camera_link, mass 0.02; collision sphere radius=0.02; visual sphere radius=0.02
- added link camera_link_optical, mass 0.0001
- added link camera_pole_link, mass 0.05; collision cylinder length=0.25 radius=0.01; visual cylinder length=0.25 radius=0.01
Joints:
- added joint camera_fixed: type fixed, parent camera_pole_link, child camera_link, origin xyz=0 0 0.125 rpy=0 -0.523 3.14159
- added joint camera_optical_joint: type fixed, parent camera_link, child camera_link_optical, origin xyz=0 0 0 rpy=-1.5708 0 -1.5708
- added joint camera_pole_fixed: type fixed, parent base_link, child camera_pole_link, origin xyz=-0.08 0.00 0.265 rpy=0 0 0

Commit message: facial recognition sensitivity fix

File: iam_bot/urdf/iam_bot.urdf (robot description, URDF)
Before this commit: robot iam_bot, 11 links, 10 joints
Links:
- link camera_pole_link: geometry collision cylinder length=0.08 radius=0.01; visual cylinder length=0.08 radius=0.01
Joints:
- joint camera_fixed: origin xyz=0 0 0.125 rpy=0 -0.523 3.14159 -> xyz=0 0 0.04 rpy=0 -0.4 3.14159
- joint camera_pole_fixed: origin xyz=-0.08 0.00 0.265 rpy=0 0 0 -> xyz=-0.08 0.00 0.18 rpy=0 0 0

Commit message: camera mapping issue fix - lidar range -5 degrees to miss cam pole

File: iam_bot/urdf/iam_bot.urdf (robot description, URDF)
Before this commit: robot iam_bot, 11 links, 10 joints
Joints:
- joint top_lidar_Rigid: origin xyz=-0.24983935 8.79e-06 0.14008005 rpy=0.0 -0.0 0.0 -> xyz=-0.24983935 8.79e-06 0.14008005 rpy=0 0 3.14159

Commit message: wheel rotation swap fix

File: iam_bot/urdf/iam_bot.urdf (robot description, URDF)
Before this commit: robot iam_bot, 11 links, 10 joints
Joints:
- joint left_wheel_Revolute: axis 0.0 0.0 1.0 -> 0.0 0.0 -1.0
- joint right_wheel_Revolute: axis 0.0 0.0 -1.0 -> 0.0 0.0 1.0

Commit message: slam navigation functional - turning halfway there

File: iam_bot/urdf/iam_bot.urdf (robot description, URDF)
Before this commit: robot iam_bot, 11 links, 10 joints
Joints:
- joint left_wheel_Revolute: axis 0.0 0.0 -1.0 -> 0.0 0.0 1.0

Commit message: map spawning attempt

File: iam_bot/urdf/iam_bot.urdf (robot description, URDF)
Before this commit: robot iam_bot, 11 links, 10 joints
Joints:
- joint right_wheel_Revolute: axis 0.0 0.0 1.0 -> 0.0 0.0 -1.0

Commit message: URDF fix - axis flip so navigation functions correctly

File: iam_bot/urdf/iam_bot.urdf (robot description, URDF)
Before this commit: robot iam_bot, 11 links, 10 joints
Links:
- link base_link: mass 2.072741935105781 -> 2.0727419351057805
- link left_wheel: mass 0.22391054430731744 -> 0.5599991469099156
- link right_wheel: mass 0.22391054430278606 -> 0.559999146909916
Joints:
- removed joint left_caster_Revolute
- removed joint left_caster_wheel_Revolute
- removed joint left_wheel_Revolute
- removed joint right_caster_Revolute
- removed joint right_caster_wheel_Revolute
- removed joint right_wheel_Revolute
- removed joint top_lidar_Rigid
- added joint left_caster_connector_revolute: type continuous, parent base_link, child left_caster_connector, origin xyz=0.07619571 0.07233422 0.02858005 rpy=3.141592653589793 -0.0 0.0, axis 0.0 0.0 1.0
- added joint left_caster_wheel_revolute: type continuous, parent left_caster_connector, child left_caster_wheel, origin xyz=-0.008249359999999992 -0.00375 0.014519849999999999 rpy=1.5707963267948966 -0.0 8.49445851048923e-121, axis 8.49445851048923e-121 0.0 -1.0
- added joint left_wheel_revolute: type continuous, parent base_link, child left_wheel, origin xyz=-0.16448079000000002 0.13288779 0.055330050000000006 rpy=-1.5707963267948968 -0.0 0.0, axis 0.0 -2.2204460492503126e-16 1.0
- added joint right_caster_connector_revolute: type continuous, parent base_link, child right_caster_connector, origin xyz=0.07619571 -0.06266578 0.02858005 rpy=3.141592653589793 -0.0 0.0, axis 0.0 0.0 1.0
- added joint right_caster_wheel_revolute: type continuous, parent right_caster_connector, child right_caster_wheel, origin xyz=-0.008249359999999992 -0.00375 0.014519849999999999 rpy=1.5707963267948966 1.5557538194652854e-61 -2.465190328815662e-32, axis -2.465190328815662e-32 3.454467422037821e-77 -1.0
- added joint right_wheel_revolute: type continuous, parent base_link, child right_wheel, origin xyz=-0.16448079000000002 -0.1367206 0.055330050000000006 rpy=1.5707963267948966 -0.0 0.0, axis 0.0 0.0 -1.0
- added joint top_lidar_fixed: type fixed, parent base_link, child top_lidar_sensor, origin xyz=0.12119571000000001 0.00233422 0.14008005 rpy=0.0 -0.0 0.0

Commit message: camera facing back of robot fix

File: iam_bot/urdf/iam_bot.urdf (robot description, URDF)
Before this commit: robot iam_bot, 11 links, 10 joints
Joints:
- joint camera_fixed: origin xyz=0 0 0.04 rpy=0 -0.4 3.14159 -> xyz=0 0 0.04 rpy=0 -0.4 0

Commit message: link removal

File: iam_bot/urdf/iam_bot.urdf (robot description, URDF)
Before this commit: robot iam_bot, 11 links, 10 joints
Links:
- removed link camera_link_optical

Commit message: camera link added

File: iam_bot/urdf/iam_bot.urdf (robot description, URDF)
Before this commit: robot iam_bot, 10 links, 10 joints
Links:
- added link camera_link_optical, mass 0.0001
